File: HMTRPBreakoutModule.sch (EAGLE design)
At the start: 23 parts, among them IC1 EUP3476, J1 Interface, J2 Flow, J3 Output, J4 Power In, Q1 DMP2035U-7

Commit message: foo
Parts:
- removed C4: 10uF, freetronics-jon:C-EUC1206
- removed C5: 2.2nF, freetronics-master-v1:CAP0603
- removed C6: 100nF, freetronics-master-v1:CAP0603
- removed D1: SK34A-LTP, freetronics-master-v1:DIODESMA
- removed D2: SS16, freetronics-jon:DIODESMAB
- removed L1: 6.8 uH, freetronics-luke:INDUCTOR
- removed LED1: Power, freetronics-master-v1:LED0603
- removed Q1: DMP2035U-7, freetronics-luke:DMP2035U-7
- removed R3: 15kΩ, freetronics-master-v1:RESISTOR0603
- removed R4: 53.6kΩ 1%, freetronics-master-v1:RESISTOR0603
- removed R5: 10kΩ, freetronics-master-v1:RESISTOR0603
- removed R6: 10kΩ 1%, freetronics-master-v1:RESISTOR0603
- added IC2: MIC5219-3.3YM5, SparkFun:V_REG_LDOSMD
- added JP1, JP2: FIDUCIAL1X2, SparkFun:FIDUCIAL1X2
- C1: value 10nF -> 2.2µF
- C2: value 22uF -> 2.2µF; device freetronics-jon:C-EUC1206 -> freetronics-master-v1:CAP0603; PACKAGE 1206 -> 0603; VOLTAGE 10V -> (none)
- C3: value 1µF -> 470pF
- IC1: value EUP3476 -> HM-TRP; device freetronics-luke:EUP3476 -> 3DRobotics:HM-TRPSMD; PACKAGE 8-SOIC -> (none)
- J2: value Flow -> Regulator Bypass; device freetronics-master-v1:M02PTH -> freetronics-luke:SJ
- J3: value Output -> Antenna; device con-molex:22-23-2061 -> 3DRobotics:SMA_EDGE
- J4: value Power In -> Config; device freetronics-master-v1:M023.5MM -> freetronics-luke:SJ
- R2: value 1kΩ -> 10kΩ
Connections:
- removed net !ENABLE: J1-2.S, Q1.G, R1.1
- removed net CTS: J2.2, J3-5.S
- removed net N$1: D2.A, J4.1
- removed net N$18: C1.1, IC1.SW, L1.1
- removed net N$19: C1.2, IC1.BS
- removed net N$2: IC1.EN, Q1.D, R5.1
- removed net N$20: C5.2, R3.2
- removed net N$21: IC1.COMP, R3.1
- removed net N$22: C6.2, IC1.SS
- removed net N$23: IC1.FB, R4.1, R6.1
- removed net N$3: LED1.A, R2.2
- removed net N$5: C2.1, D1.A, L1.2, R4.2
- removed net RTS: J2.1, J3-1.S
- removed net RXD: J1-4.S, J3-3.S
- removed net TXD: J1-3.S, J3-2.S
- removed net VIN: C4.1, D2.C, IC1.IN, Q1.S
- new net +3V3: C2.1, IC1.VCC, IC2.OUT, J2.2, R1.1
- new net N$11: IC1.DRX, J1-4.S
- new net N$13: C3.2, IC2.BP
- new net N$14: IC1.!CONFIG, J4.2, R1.2
- new net N$6: IC1.!ENABLE, J1-2.S, R2.1
- new net N$7: IC1.DTX, J1-3.S
- new net N$8: IC1.ANT, J3.SIGNAL
- net +5V: now also C1.1, IC2.EN, IC2.IN, J1-1.S, J2.1; no longer C3.2, D1.C, J3-4.S, R2.1
- net GND: now also C1.2, IC1.AGND, IC2.GND, J3.GND@0, J3.GND@1, J3.GND@2, J3.GND@3, J4.1, R2.2; no longer C4.2, C5.1, C6.1, IC1.TGND, J3-6.S, J4.2, LED1.C, R1.2, R5.2, R6.2
Other:
- note added: "GROUND"
- note added: "HM-TRP Radio Module Breakout Board"
- note removed: "+5V"
- note removed: "CTS"
- note removed: "GND"
- note removed: "Ground"
- note removed: "RFD900 UHF Modem Power Supply Module"
- note removed: "RTS"
- moved on the sheet: C1, C2, C3, J1-1, J1-2, J1-3, J1-4, J1-5, R1, R2
