File: HighRangeAccelerometer.brd (EAGLE design)
At the start: 24.2 x 21.6 mm, 11 parts, among them IC1 MCP3202-CI/SN, IC2 AD22282-A-R2, J1 Interface, J2 Self-test

Commit message: foo
Parts:
- removed R1: 10kΩ, freetronics-master-v1:0603
- moved C2 28.7 mm to (18.4, 19.7)
- moved IC1 28.7 mm to (8.89, 14.0)
- moved IC2 28.7 mm to (15.9, 15.2)
- moved J1 28.7 mm to (12.7, 5.08)
- moved J2 28.7 mm to (17.1, 10.2)
- moved LED1 28.7 mm to (16.5, 7.94)
- moved R2 28.7 mm to (19.7, 7.94)
- moved C3 28.7 mm to (15.2, 19.7)
- moved C1 28.4 mm to (13.3, 10.8)
- moved SY 27.0 mm to (22.9, 6.99)
Connections:
- net +5V: no longer R1.2
- net N$23: no longer R1.1
Routing:
- net +5V: track 50.0 -> 38.3 mm, vias 4 -> 2
- net GND: track 6.12 -> 3.95 mm
- net N$23: track 28.6 -> 27.5 mm
Other:
- board size 24.2 x 21.6 mm -> 24.2 x 22.2 mm
- board text added: "!CS"
- board text added: "+Ax"
- board text added: "Luke Weston, 2013"
- board text removed: "."
- board text removed: "/CS"
- board text removed: "LED"
- board text removed: "Luke Weston, 2011"
- board text removed: "accelerometery axis"
- board text removed: "self-test"

Commit message: foo
Parts:
- J1: value Interface -> Self-test; device con-molex:7395-06 -> jumper:SJ
- J2: value Self-test -> Interface; device jumper:SJ -> con-molex:22-23-2061
- moved J2 8.28 mm to (12.7, 3.17), flipped to the top
- moved J1 6.75 mm to (17.1, 10.2), flipped to the bottom
- renumbered LED1 to LED, R2 to R1
Connections:
- net +5V: now also J1.2, J2.6; no longer J1.1, J2.2
- net GND: now also J2.5; no longer J1.2
- net N$18: now also J2.4; no longer J1.3
- net N$21: now also J2.3; no longer J1.4
- net N$22: now also J2.2; no longer J1.5
- net N$23: now also J2.1; no longer J1.6
- net N$25: now also J1.1; no longer J2.1
Routing:
- net N$23: track 27.5 -> 29.5 mm
- net +5V: track 38.3 -> 40.2 mm
- net N$22: track 11.2 -> 12.8 mm
Other:
- board size 24.2 x 22.2 mm -> 24.2 x 23.5 mm
