File: HighRangeAccelerometer.sch (EAGLE design)
At the start: 11 parts, among them IC1 MCP3202-CI/SN, IC2 AD22282-A-R2, J1 Interface, J2 Self-test

Commit message: foo
Parts:
- removed R1: 10kΩ, freetronics-master-v1:RESISTOR0603
Connections:
- net +5V: no longer R1.2
- net N$23: no longer R1.1
Changed lines of the file:
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@@
 <attribute name="PACKAGE" value="0603"/>
 </part>
-<part name="R1" library="freetronics-master-v1" deviceset="RESISTOR" device="0603" value="10kΩ">
-<attribute name="PACKAGE" value="0603"/>
-</part>
-<part name="U$2" library="freetronics-luke" deviceset="+5V" device=""/>
 <part name="J2" library="jumper" deviceset="SJ" device="" value="Self-test"/>
 <part name="U$3" library="freetronics-luke" deviceset="+5V" device=""/>
@@
 <attribute name="PACKAGE" x="144.78" y="83.82" size="1.27" layer="96"/>
 </instance>
-<instance part="R1" gate="G$1" x="86.36" y="111.76" smashed="yes" rot="R90">
-<attribute name="NAME" x="78.74" y="114.3" size="1.27" layer="95"/>
-<attribute name="VALUE" x="78.74" y="111.76" size="1.27" layer="96"/>
-<attribute name="PACKAGE" x="78.74" y="109.22" size="1.27" layer="96"/>
-</instance>
-<instance part="U$2" gate="G$1" x="86.36" y="121.92"/>
 <instance part="J2" gate="1" x="162.56" y="101.6" smashed="yes" rot="MR90">
 <attribute name="NAME" x="165.1" y="101.6" size="1.27" layer="95"/>
@@
 <wire x1="91.44" y1="104.14" x2="101.6001" y2="104.14" width="0.1524" layer="91"/>
 <wire x1="91.44" y1="91.44" x2="91.44" y2="104.14" width="0.1524" layer="91"/>
-</segment>
-<segment>
-<pinref part="R1" gate="G$1" pin="2"/>
-<pinref part="U$2" gate="G$1" pin="+5V"/>
-<wire x1="86.36" y1="119.38" x2="86.36" y2="116.84" width="0.1524" layer="91"/>
 </segment>
 <segment>
@@
 <wire x1="86.36" y1="96.52" x2="101.6001" y2="96.52" width="0.1524" layer="91"/>
 <pinref part="IC1" gate="P" pin="!CS!/SHDN"/>
-<pinref part="R1" gate="G$1" pin="1"/>
-<wire x1="86.36" y1="106.68" x2="86.36" y2="96.52" width="0.1524" layer="91"/>
-<junction x="86.36" y="96.52"/>
-</segment>
-</net>
+</segment>
+</net>

Commit message: foo
Parts:
- J1: value Interface -> Self-test; device con-molex:22-05-7068-06 -> jumper:SJ
- J2: value Self-test -> Interface; device jumper:SJ -> con-molex:22-23-2061
- renumbered LED1 to LED, R2 to R1
Connections:
- net +5V: now also J1.2, J2-6.S; no longer J1-1.S, J2.2
- net GND: now also J2-5.S; no longer J1-2.S
- net N$18: now also J2-4.S; no longer J1-3.S
- net N$21: now also J2-3.S; no longer J1-4.S
- net N$22: now also J2-2.S; no longer J1-5.S
- net N$23: now also J2-1.S; no longer J1-6.S
- net N$25: now also J1.1; no longer J2.1
Other:
- note added: "!CS"
- note added: "GND"
- note added: "MISO"
- note added: "MOSI"
- note added: "SCK"
- note added: "VCC"
Changed lines of the file:
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@@
 <part name="FRAME2" library="frames" deviceset="A4L-LOC" device="" value="Frame1"/>
 <part name="SY" library="SparkFun" deviceset="OSHW-LOGO" device="S"/>
-<part name="J1" library="con-molex" deviceset="22-?-06" device="05-7068" value="Interface"/>
 <part name="U$1" library="freetronics-luke" deviceset="+5V" device=""/>
 <part name="G1" library="freetronics-luke" deviceset="GND" device=""/>
@@
 <attribute name="PACKAGE" value="0603"/>
 </part>
-<part name="J2" library="jumper" deviceset="SJ" device="" value="Self-test"/>
+<part name="J1" library="jumper" deviceset="SJ" device="" value="Self-test"/>
 <part name="U$3" library="freetronics-luke" deviceset="+5V" device=""/>
 <part name="U$4" library="freetronics-luke" deviceset="+5V" device=""/>
 <part name="G7" library="freetronics-luke" deviceset="GND" device=""/>
-<part name="LED1" library="freetronics-master-v1" deviceset="LED" device="0603" value="Power">
+<part name="LED" library="freetronics-master-v1" deviceset="LED" device="0603" value="Power">
 <attribute name="COLOUR" value="Blue"/>
 <attribute name="PACKAGE" value="0603"/>
@@
 </part>
 <part name="G8" library="freetronics-luke" deviceset="GND" device=""/>
-<part name="R2" library="freetronics-master-v1" deviceset="RESISTOR" device="0603" value="1kΩ">
+<part name="R1" library="freetronics-master-v1" deviceset="RESISTOR" device="0603" value="1kΩ">
 <attribute name="PACKAGE" value="0603"/>
 </part>
 <part name="G9" library="freetronics-luke" deviceset="GND" device=""/>
 <part name="U$5" library="freetronics-luke" deviceset="+5V" device=""/>
+<part name="J2" library="con-molex" deviceset="22-23-2061" device="" value="Interface"/>
 </parts>
 <sheets>
@@
 <text x="15.24" y="12.7" size="2.1844" layer="97">Released under the CERN Open Hardware License:</text>
 <text x="35.56" y="7.62" size="2.1844" layer="97">http://ohwr.org/cernohl</text>
+<text x="58.42" y="103.632" size="1.27" layer="97">VCC</text>
+<text x="58.42" y="101.092" size="1.27" layer="97">GND</text>
+<text x="58.42" y="98.552" size="1.27" layer="97">MISO</text>
+<text x="58.42" y="96.012" size="1.27" layer="97">MOSI</text>
+<text x="58.42" y="93.472" size="1.27" layer="97">SCK</text>
+<text x="58.42" y="90.932" size="1.27" layer="97">!CS</text>
 </plain>
 <instances>
 <instance part="FRAME2" gate="G$1" x="0" y="0"/>
 <instance part="SY" gate="G$1" x="129.54" y="17.78" smashed="yes"/>
-<instance part="J1" gate="-1" x="71.12" y="104.14" smashed="yes" rot="R180">
-<attribute name="NAME" x="63.5" y="104.14" size="1.27" layer="95"/>
-<attribute name="VALUE" x="71.12" y="106.68" size="1.27" layer="96"/>
-</instance>
-<instance part="J1" gate="-2" x="71.12" y="101.6" smashed="yes" rot="R180">
-<attribute name="NAME" x="63.5" y="101.6" size="1.27" layer="95"/>
-</instance>
-<instance part="J1" gate="-3" x="71.12" y="99.06" smashed="yes" rot="R180">
-<attribute name="NAME" x="63.5" y="99.06" size="1.27" layer="95"/>
-</instance>
-<instance part="J1" gate="-4" x="71.12" y="96.52" smashed="yes" rot="R180">
-<attribute name="NAME" x="63.5" y="96.52" size="1.27" layer="95"/>
-</instance>
-<instance part="J1" gate="-5" x="71.12" y="93.98" smashed="yes" rot="R180">
-<attribute name="NAME" x="63.5" y="93.98" size="1.27" layer="95"/>
-</instance>
-<instance part="J1" gate="-6" x="71.12" y="91.44" smashed="yes" rot="R180">
-<attribute name="NAME" x="63.5" y="91.44" size="1.27" layer="95"/>
-</instance>
 <instance part="U$1" gate="G$1" x="91.44" y="109.22"/>
 <instance part="G1" gate="G$1" x="76.2" y="78.74" rot="MR0"/>
@@
 <attribute name="PACKAGE" x="144.78" y="83.82" size="1.27" layer="96"/>
 </instance>
-<instance part="J2" gate="1" x="162.56" y="101.6" smashed="yes" rot="MR90">
+<instance part="J1" gate="1" x="162.56" y="101.6" smashed="yes" rot="MR90">
 <attribute name="NAME" x="165.1" y="101.6" size="1.27" layer="95"/>
 <attribute name="VALUE" x="165.1" y="99.06" size="1.27" layer="96"/>
@@
 <instance part="U$4" gate="G$1" x="154.94" y="109.22"/>
 <instance part="G7" gate="G$1" x="154.94" y="78.74" rot="MR0"/>
-<instance part="LED1" gate="G$1" x="177.8" y="88.9" smashed="yes" rot="MR0">
+<instance part="LED" gate="G$1" x="177.8" y="88.9" smashed="yes" rot="MR0">
 <attribute name="NAME" x="182.88" y="88.9" size="1.27" layer="95"/>
 <attribute name="VALUE" x="182.88" y="86.36" size="1.27" layer="96"/>
@@
 </instance>
 <instance part="G8" gate="G$1" x="167.64" y="78.74" rot="MR0"/>
-<instance part="R2" gate="G$1" x="177.8" y="99.06" smashed="yes" rot="R90">
+<instance part="R1" gate="G$1" x="177.8" y="99.06" smashed="yes" rot="R90">
 <attribute name="NAME" x="180.34" y="101.6" size="1.27" layer="95"/>
 <attribute name="VALUE" x="180.34" y="99.06" size="1.27" layer="96"/>
@@
 <instance part="G9" gate="G$1" x="177.8" y="78.74" rot="MR0"/>
 <instance part="U$5" gate="G$1" x="177.8" y="109.22"/>
+<instance part="J2" gate="-1" x="71.12" y="91.44" smashed="yes" rot="R180">
+<attribute name="NAME" x="63.5" y="90.678" size="1.524" layer="95"/>
+<attribute name="VALUE" x="68.58" y="106.68" size="1.27" layer="96"/>
+</instance>
+<instance part="J2" gate="-2" x="71.12" y="93.98" smashed="yes" rot="R180">
+<attribute name="NAME" x="63.5" y="93.218" size="1.524" layer="95"/>
+</instance>
+<instance part="J2" gate="-3" x="71.12" y="96.52" smashed="yes" rot="R180">
+<attribute name="NAME" x="63.5" y="95.758" size="1.524" layer="95"/>
+</instance>
+<instance part="J2" gate="-4" x="71.12" y="99.06" smashed="yes" rot="R180">
+<attribute name="NAME" x="63.5" y="98.298" size="1.524" layer="95"/>
+</instance>
+<instance part="J2" gate="-5" x="71.12" y="101.6" smashed="yes" rot="R180">
+<attribute name="NAME" x="63.5" y="100.838" size="1.524" layer="95"/>
+</instance>
+<instance part="J2" gate="-6" x="71.12" y="104.14" smashed="yes" rot="R180">
+<attribute name="NAME" x="63.5" y="103.378" size="1.524" layer="95"/>
+</instance>
 </instances>
 <busses>
@@
 <net name="+5V" class="0">
 <segment>
-<pinref part="J1" gate="-1" pin="S"/>
 <wire x1="73.66" y1="104.14" x2="91.44" y2="104.14" width="0.1524" layer="91"/>
 <pinref part="U$1" gate="G$1" pin="+5V"/>
@@
 <wire x1="91.44" y1="104.14" x2="101.6001" y2="104.14" width="0.1524" layer="91"/>
 <wire x1="91.44" y1="91.44" x2="91.44" y2="104.14" width="0.1524" layer="91"/>
-</segment>
-<segment>
-<pinref part="J2" gate="1" pin="2"/>
+<pinref part="J2" gate="-6" pin="S"/>
+</segment>
+<segment>
+<pinref part="J1" gate="1" pin="2"/>
 <pinref part="U$3" gate="G$1" pin="+5V"/>
 <wire x1="162.56" y1="106.68" x2="162.56" y2="104.14" width="0.1524" layer="91"/>
@@
 </segment>
 <segment>
-<pinref part="R2" gate="G$1" pin="2"/>
+<pinref part="R1" gate="G$1" pin="2"/>
 <pinref part="U$5" gate="G$1" pin="+5V"/>
 <wire x1="177.8" y1="106.68" x2="177.8" y2="104.14" width="0.1524" layer="91"/>
@@
 <net name="GND" class="0">
 <segment>
-<pinref part="J1" gate="-2" pin="S"/>
 <wire x1="73.66" y1="101.6" x2="76.2" y2="101.6" width="0.1524" layer="91"/>
 <pinref part="G1" gate="G$1" pin="GND"/>
 <wire x1="76.2" y1="101.6" x2="76.2" y2="81.28" width="0.1524" layer="91"/>
+<pinref part="J2" gate="-5" pin="S"/>
 </segment>
 <segment>
@@
 </segment>
 <segment>
-<pinref part="LED1" gate="G$1" pin="C"/>
+<pinref part="LED" gate="G$1" pin="C"/>
 <pinref part="G9" gate="G$1" pin="GND"/>
 <wire x1="177.8" y1="81.28" x2="177.8" y2="83.82" width="0.1524" layer="91"/>
@@
 <wire x1="101.6001" y1="93.98" x2="81.28" y2="93.98" width="0.1524" layer="91"/>
 <wire x1="81.28" y1="93.98" x2="81.28" y2="99.06" width="0.1524" layer="91"/>
-<pinref part="J1" gate="-3" pin="S"/>
 <wire x1="81.28" y1="99.06" x2="73.66" y2="99.06" width="0.1524" layer="91"/>
 <pinref part="IC1" gate="P" pin="DOUT"/>
+<pinref part="J2" gate="-4" pin="S"/>
 </segment>
 </net>
 <net name="N$21" class="0">
 <segment>
-<pinref part="J1" gate="-4" pin="S"/>
 <wire x1="73.66" y1="96.52" x2="83.82" y2="96.52" width="0.1524" layer="91"/>
 <wire x1="83.82" y1="96.52" x2="83.82" y2="99.06" width="0.1524" layer="91"/>
 <wire x1="83.82" y1="99.06" x2="101.6001" y2="99.06" width="0.1524" layer="91"/>
 <pinref part="IC1" gate="P" pin="DIN"/>
+<pinref part="J2" gate="-3" pin="S"/>
 </segment>
 </net>
 <net name="N$22" class="0">
 <segment>
-<pinref part="J1" gate="-5" pin="S"/>
 <wire x1="73.66" y1="93.98" x2="78.74" y2="93.98" width="0.1524" layer="91"/>
 <wire x1="78.74" y1="93.98" x2="78.74" y2="101.6" width="0.1524" layer="91"/>
 <wire x1="78.74" y1="101.6" x2="101.6001" y2="101.6" width="0.1524" layer="91"/>
 <pinref part="IC1" gate="P" pin="CLK"/>
+<pinref part="J2" gate="-2" pin="S"/>
 </segment>
 </net>
 <net name="N$23" class="0">
 <segment>
-<pinref part="J1" gate="-6" pin="S"/>
 <wire x1="73.66" y1="91.44" x2="86.36" y2="91.44" width="0.1524" layer="91"/>
 <wire x1="86.36" y1="91.44" x2="86.36" y2="96.52" width="0.1524" layer="91"/>
 <wire x1="86.36" y1="96.52" x2="101.6001" y2="96.52" width="0.1524" layer="91"/>
 <pinref part="IC1" gate="P" pin="!CS!/SHDN"/>
+<pinref part="J2" gate="-1" pin="S"/>
 </segment>
 </net>
@@
 <pinref part="IC2" gate="G$1" pin="ST"/>
 <wire x1="152.4" y1="96.52" x2="162.56" y2="96.52" width="0.1524" layer="91"/>
-<pinref part="J2" gate="1" pin="1"/>
+<pinref part="J1" gate="1" pin="1"/>
 <wire x1="162.56" y1="96.52" x2="162.56" y2="99.06" width="0.1524" layer="91"/>
 </segment>
@@
 <net name="N$12" class="0">
 <segment>
-<pinref part="LED1" gate="G$1" pin="A"/>
-<pinref part="R2" gate="G$1" pin="1"/>
+<pinref part="LED" gate="G$1" pin="A"/>
+<pinref part="R1" gate="G$1" pin="1"/>
 <wire x1="177.8" y1="93.98" x2="177.8" y2="91.44" width="0.1524" layer="91"/>
 </segment>
