File: RFD900module.brd (EAGLE design)
At the start: 50.8 x 31.8 mm, 21 parts, among them IC1 EUP3476, J1 Flow, J2 Interface, J3 Power In, J4 RFD900 RF Modem

Commit message: foo
Parts:
- added Q1: DMP2035U-7, freetronics-luke:SOT23-3
- added R6: 10kΩ 1%, freetronics-master-v1:0603
- J1: value Flow -> Interface; device freetronics-master-v1:1X02 -> con-molex:22-23-2051
- J2: value Interface -> Flow; device con-molex:7395-04 -> freetronics-master-v1:1X02
- J3: value Power In -> Output; device freetronics-master-v1:SCREWTERMINAL-3.5MM-2 -> con-molex:22-23-2061
- J4: value RFD900 RF Modem -> Power In; device con-molex:7395-06 -> freetronics-master-v1:SCREWTERMINAL-3.5MM-2
- R1: value 100kΩ -> 10kΩ
- R5: value 10kΩ 1% -> 10kΩ
- moved J3 46.8 mm to (52.1, 17.8), turned to 90 degrees
- moved J4 41.9 mm to (6.35, 27.9), turned to 270 degrees
- moved J2 11.1 mm to (9.53, 5.08), turned to 180 degrees
- moved R1 11.0 mm to (14.6, 28.6), turned to 180 degrees
- moved R5 10.9 mm to (17.5, 25.4), turned to 180 degrees
- moved J1 9.09 mm to (6.99, 14.0), turned to 270 degrees
- moved SY 1.27 mm to (48.3, 5.08)
Connections:
- removed net EN: IC1.7, J2.1, R1.1
- new net !ENABLE: J1.2, Q1.1, R1.1
- new net N$2: IC1.7, Q1.3, R5.1
- net +5V: now also J3.4; no longer J4.3
- net CTS: now also J2.2, J3.5; no longer J1.2, J4.2
- net GND: now also J1.5, J3.6, J4.2, R1.2, R6.2; no longer J2.4, J3.2, J4.1
- net N$1: now also J4.1; no longer J3.1
- net N$23: now also R6.1; no longer R5.1
- net RTS: now also J2.1, J3.1; no longer J1.1, J4.6
- net RXD: now also J1.4, J3.3; no longer J2.3, J4.4
- net TXD: now also J1.3, J3.2; no longer J2.2, J4.5
- net VIN: now also Q1.2; no longer R1.2
Routing:
- net EN: track 31.4 -> 0.00 mm, vias 3 -> 0
- net !ENABLE: track 0.00 -> 23.4 mm, vias 0 -> 1
- net VIN: track 16.2 -> 27.9 mm, vias 0 -> 2
- net TXD: track 43.0 -> 54.6 mm, vias 1 -> 0
- net N$2: track 0.00 -> 10.9 mm
- net CTS: track 47.7 -> 54.0 mm, vias 0 -> 1
- net +5V: track 9.74 -> 14.8 mm
- net RXD: track 44.0 -> 47.2 mm
- net RTS: track 44.5 -> 45.2 mm
Other:
- board size 50.8 x 31.8 mm -> 55.9 x 31.8 mm
- board text added: "!EN"
- board text added: "+5VOut"
- board text added: "CTS"
- board text added: "GND"
- board text added: "Luke Weston, 2013"
- board text added: "NC"
- board text added: "RFD900 RF Modem Power Supply / Breakout Board"
- board text added: "RTS"
- board text added: "RXD"
- board text added: "TXD"
