File: FGPMMOPA6x.brd (EAGLE design)
At the start: 26 x 33.7 mm, 13 parts, among them IC1 FGPMMOPA6H, J1 PPS, J2 Interface, J3 U.FL

Commit message: foo
Parts:
- removed SY2: OSHW-LOGOS, SparkFun:OSHW-LOGO-S
- added SY: OSHW-LOGOS, SparkFun:OSHW-LOGO-S
- J2: device con-molex:7395-04 -> con-molex:22-23-2041
- LED2: value GPS Status -> Status
- moved J2 1.27 mm to (11.4, 7.62)
Connections:
- net +3V3: now also J2.4; no longer J2.1
- net GND: now also J2.3; no longer J2.2
- net N$14: now also J2.1; no longer J2.4
- net N$15: now also J2.2; no longer J2.3
Routing:
- net N$15: track 40.0 -> 38.7 mm
- net +3V3: track 31.3 -> 31.9 mm
- net N$14: track 44.0 -> 43.5 mm
Other:
- board text added: "+ Side Up"
- board text added: "+3.3"
- board text added: "CR1220 12mm 3V Cell"
- board text removed: "+3.3V"
