File: FGPMMOPA6x.sch (EAGLE design)
At the start: 13 parts, among them IC1 FGPMMOPA6H, J1 PPS, J2 Interface, J3 U.FL

Commit message: foo
Parts:
- C1: PACKAGE 0603 -> 0805
Changed lines of the file:
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@@
 </part>
 <part name="C1" library="freetronics-master-v1" deviceset="CAP" device="0805" value="10µF">
-<attribute name="PACKAGE" value="0603"/>
+<attribute name="PACKAGE" value="0805"/>
 </part>
 <part name="G14" library="freetronics-luke" deviceset="GND" device=""/>

Commit message: foo
Parts:
- J2: device con-molex:22-05-7048-04 -> con-molex:22-23-2041; OC_FARNELL unknown -> (none); OC_NEWARK unknown -> (none)
- LED2: value GPS Status -> Status
- renumbered SY2 to SY
Connections:
- net +3V3: now also J2-4.S; no longer J2-1.S
- net GND: now also J2-3.S; no longer J2-2.S
- net N$14: now also J2-1.S; no longer J2-4.S
- net N$15: now also J2-2.S; no longer J2-3.S
Other:
- note added: "+3.3V"
- note added: "GND"
- note added: "RXD"
- note added: "TXD"
- moved on the sheet: J2-1, J2-2, J2-3, J2-4
Changed lines of the file:
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@@
 <setting verticaltext="up"/>
 </settings>
-<grid distance="0.1" unitdist="inch" unit="inch" style="lines" multiple="1" display="no" altdistance="0.01" altunitdist="inch" altunit="inch"/>
+<grid distance="0.1" unitdist="inch" unit="inch" style="lines" multiple="1" display="yes" altdistance="0.01" altunitdist="inch" altunit="inch"/>
 <layers>
 <layer number="1" name="Top" color="4" fill="1" visible="no" active="no"/>
@@
 <part name="G11" library="freetronics-luke" deviceset="GND" device=""/>
 <part name="G12" library="freetronics-luke" deviceset="GND" device=""/>
-<part name="LED2" library="freetronics-master-v1" deviceset="LED" device="0603" value="GPS Status">
+<part name="LED2" library="freetronics-master-v1" deviceset="LED" device="0603" value="Status">
 <attribute name="COLOUR" value="Yellow"/>
 <attribute name="PACKAGE" value="0603"/>
@@
 </part>
 <part name="U$41" library="freetronics-luke" deviceset="+3.3V" device=""/>
-<part name="J2" library="con-molex" deviceset="22-?-04" device="05-7048" value="Interface">
-<attribute name="MF" value=""/>
-<attribute name="MPN" value=""/>
-<attribute name="OC_FARNELL" value="unknown"/>
-<attribute name="OC_NEWARK" value="unknown"/>
-</part>
 <part name="U$39" library="freetronics-luke" deviceset="+3.3V" device=""/>
 <part name="G16" library="freetronics-luke" deviceset="GND" device=""/>
@@
 <part name="U$42" library="freetronics-luke" deviceset="+3.3V" device=""/>
 <part name="B1" library="SparkFun" deviceset="BATTERY" device="12MM" value="Keystone 3000"/>
-<part name="SY2" library="SparkFun" deviceset="OSHW-LOGO" device="S"/>
+<part name="SY" library="SparkFun" deviceset="OSHW-LOGO" device="S"/>
+<part name="J2" library="con-molex" deviceset="22-23-2041" device="" value="Interface"/>
 </parts>
 <sheets>
@@
 <text x="15.24" y="12.7" size="2.1844" layer="97">Released under the CERN Open Hardware License:</text>
 <text x="35.56" y="7.62" size="2.1844" layer="97">http://ohwr.org/cernohl</text>
+<text x="45.72" y="88.9" size="1.27" layer="97">+3.3V</text>
+<text x="45.72" y="86.36" size="1.27" layer="97">GND</text>
+<text x="45.72" y="83.82" size="1.27" layer="97">RXD</text>
+<text x="45.72" y="81.28" size="1.27" layer="97">TXD</text>
 </plain>
 <instances>
@@
 </instance>
 <instance part="U$41" gate="G$1" x="132.08" y="129.54" rot="MR0"/>
-<instance part="J2" gate="-1" x="60.96" y="88.9" smashed="yes" rot="MR0">
-<attribute name="NAME" x="53.34" y="88.9" size="1.27" layer="95"/>
-<attribute name="VALUE" x="53.34" y="91.44" size="1.27" layer="96"/>
-</instance>
-<instance part="J2" gate="-2" x="60.96" y="86.36" smashed="yes" rot="MR0">
-<attribute name="NAME" x="53.34" y="86.36" size="1.27" layer="95"/>
-</instance>
-<instance part="J2" gate="-3" x="60.96" y="83.82" smashed="yes" rot="MR0">
-<attribute name="NAME" x="53.34" y="83.82" size="1.27" layer="95"/>
-</instance>
-<instance part="J2" gate="-4" x="60.96" y="81.28" smashed="yes" rot="MR0">
-<attribute name="NAME" x="53.34" y="81.28" size="1.27" layer="95"/>
-</instance>
 <instance part="U$39" gate="G$1" x="66.04" y="104.14"/>
 <instance part="G16" gate="G$1" x="66.04" y="66.04" rot="MR0"/>
@@
 <attribute name="VALUE" x="88.9" y="104.14" size="1.27" layer="96"/>
 </instance>
-<instance part="SY2" gate="G$1" x="129.54" y="17.78" smashed="yes"/>
+<instance part="SY" gate="G$1" x="129.54" y="17.78" smashed="yes"/>
+<instance part="J2" gate="-1" x="60.96" y="81.28" smashed="yes" rot="R180">
+<attribute name="NAME" x="53.34" y="80.772" size="1.27" layer="95"/>
+<attribute name="VALUE" x="53.34" y="91.44" size="1.27" layer="96"/>
+</instance>
+<instance part="J2" gate="-2" x="60.96" y="83.82" smashed="yes" rot="R180">
+<attribute name="NAME" x="53.34" y="83.312" size="1.27" layer="95"/>
+</instance>
+<instance part="J2" gate="-3" x="60.96" y="86.36" smashed="yes" rot="R180">
+<attribute name="NAME" x="53.34" y="85.852" size="1.27" layer="95"/>
+</instance>
+<instance part="J2" gate="-4" x="60.96" y="88.9" smashed="yes" rot="R180">
+<attribute name="NAME" x="53.34" y="88.392" size="1.27" layer="95"/>
+</instance>
 </instances>
 <busses>
@@
 </segment>
 <segment>
-<pinref part="J2" gate="-2" pin="S"/>
 <wire x1="63.5" y1="86.36" x2="66.04" y2="86.36" width="0.1524" layer="91"/>
 <wire x1="66.04" y1="86.36" x2="66.04" y2="68.58" width="0.1524" layer="91"/>
 <pinref part="G16" gate="G$1" pin="GND"/>
+<pinref part="J2" gate="-3" pin="S"/>
 </segment>
 <segment>
@@
 </segment>
 <segment>
-<pinref part="J2" gate="-1" pin="S"/>
 <wire x1="63.5" y1="88.9" x2="66.04" y2="88.9" width="0.1524" layer="91"/>
 <wire x1="66.04" y1="88.9" x2="66.04" y2="101.6" width="0.1524" layer="91"/>
 <pinref part="U$39" gate="G$1" pin="+3V3"/>
+<pinref part="J2" gate="-4" pin="S"/>
 </segment>
 <segment>
@@
 <pinref part="IC1" gate="G$1" pin="TX"/>
 <wire x1="144.78" y1="86.36" x2="76.2" y2="86.36" width="0.1524" layer="91"/>
-<pinref part="J2" gate="-4" pin="S"/>
 <wire x1="63.5" y1="81.28" x2="76.2" y2="81.28" width="0.1524" layer="91"/>
 <wire x1="76.2" y1="81.28" x2="76.2" y2="86.36" width="0.1524" layer="91"/>
+<pinref part="J2" gate="-1" pin="S"/>
 </segment>
 </net>
@@
 <pinref part="IC1" gate="G$1" pin="RX"/>
 <wire x1="144.78" y1="83.82" x2="63.5" y2="83.82" width="0.1524" layer="91"/>
-<pinref part="J2" gate="-3" pin="S"/>
+<pinref part="J2" gate="-2" pin="S"/>
 </segment>
 </net>
@@
 </sheet>
 </sheets>
+<errors>
+</errors>
 </schematic>
 </drawing>
