File: OEMV1_GPS_Interface.brd (EAGLE design)
At the start: 44.1 x 27.3 mm, 30 parts, among them IC1 EUP3476, IC2 SN65HVD230DR, J1 LNA Power, J2 OEMV-1 GPS Receiver, J3 USB, J4 CAN, J5 CAN Terminate, J6 UART

Commit message: foo
Parts:
- added SY: OSHW-LOGOS, SparkFun:OSHW-LOGO-S
Changed lines of the file:
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@@
 <attribute name="VALUE" x="35.8775" y="13.335" size="0.8128" layer="27" ratio="15" rot="R90"/>
 </element>
+<element name="SY" library="SparkFun" package="OSHW-LOGO-S" value="OSHW-LOGOS" x="1.905" y="-1.905"/>
 </elements>
 <signals>
