File: OEMV1_GPS_Interface.sch (EAGLE design)
At the start: 30 parts, among them IC1 EUP3476, IC2 SN65HVD230DR, J1 LNA Power, J2 OEMV-1 GPS Receiver, J3 USB, J4 CAN, J5 CAN Terminate, J6 UART

Commit message: foo
Parts:
- added SY: OSHW-LOGOS, SparkFun:OSHW-LOGOS
Changed lines of the file:
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@@
 <attribute name="VOLTAGE" value="6.3V"/>
 </part>
+<part name="SY" library="SparkFun" deviceset="OSHW-LOGO" device="S"/>
 </parts>
 <sheets>
@@
 <attribute name="VOLTAGE" x="111.76" y="106.68" size="1.27" layer="96"/>
 </instance>
+<instance part="SY" gate="G$1" x="134.62" y="20.32" smashed="yes"/>
 </instances>
 <busses>
