File: Venus638FLPX-L.brd (EAGLE design)
At the start: 38.7 x 20.3 mm, 14 parts, among them IC1 VENUS638FLPX-L, J1 Interface

Commit message: foo
Parts:
- removed JP1: Antenna, SparkFun:SMA-EDGE
- added J2: Interface, con-molex:22-23-2041
- added SY: OSHW-LOGOS, SparkFun:OSHW-LOGO-S
- J1: value Interface -> Antenna; device con-molex:7395-04 -> SparkFun:SMA-EDGE
- LED1: value GPS Status -> Status
- moved J1 21.5 mm to (36.2, 19.1), turned to 90 degrees
Connections:
- net +3.3V: now also J2.4; no longer J1.1
- net ANT2: now also J1.SIG; no longer JP1.SIG
- net GND: now also J2.3; no longer J1.2
- net RFGND: now also J1.GND@0, J1.GND@1, J1.GND@2, J1.GND@3; no longer JP1.GND@0, JP1.GND@1, JP1.GND@2, JP1.GND@3
- net RXD: now also J2.2; no longer J1.3
- net TXD: now also J2.1; no longer J1.4
Routing:
- net RXD: track 17.1 -> 20.8 mm
- net TXD: track 6.95 -> 10.5 mm
- net RFGND: track 1.62 -> 0.00 mm
- net +3.3V: track 58.1 -> 59.3 mm, vias 4 -> 3
Other:
- board size 38.7 x 20.3 mm -> 33.3 x 20.3 mm
- board text added: "+ Side Up"
- board text added: "3V3"
- board text added: "CR1220 12mm 3V Cell"
- board text added: "GND"
- board text added: "J1"
- board text added: "Luke Weston, 2013"
- board text added: "RXD"
- board text added: "TXD"
- board text added: "Venus 638FLPX-L GPS Receiver"
