File: Venus638FLPX-L.sch (EAGLE design)
At the start: 14 parts, among them IC1 VENUS638FLPX-L, J1 Interface

Commit message: foo
Parts:
- removed JP1: Antenna, SparkFun:SMA_EDGE
- added J2: Interface, con-molex:22-23-2041
- added SY: OSHW-LOGOS, SparkFun:OSHW-LOGOS
- J1: value Interface -> Antenna; device con-molex:22-05-7048-04 -> SparkFun:SMA_EDGE
- LED1: value GPS Status -> Status
Connections:
- net +3.3V: now also J2-4.S; no longer J1-1.S
- net ANT2: now also J1.SIGNAL; no longer JP1.SIGNAL
- net GND: now also J2-3.S; no longer J1-2.S
- net RFGND: now also J1.GND@0, J1.GND@1, J1.GND@2, J1.GND@3; no longer JP1.GND@0, JP1.GND@1, JP1.GND@2, JP1.GND@3
- net RXD: now also J2-2.S; no longer J1-3.S
- net TXD: now also J2-1.S; no longer J1-4.S
Other:
- note added: "Luke Weston, 2013"
- note added: "Released under the CERN Open Hardware License:"
- note added: "Venus 638FLPX-L GPS Receiver Module"
- note added: "http://github.com/lukeweston/SSRPGenericTelemetryModule"
- note added: "http://ohwr.org/cernohl"
Changed lines of the file:
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@@
 <part name="IC1" library="mike-temp" deviceset="VENUS638FLPX-L" device=""/>
 <part name="G18" library="freetronics-luke" deviceset="GND" device=""/>
-<part name="LED1" library="freetronics-master-v1" deviceset="LED" device="0603" value="GPS Status">
+<part name="LED1" library="freetronics-master-v1" deviceset="LED" device="0603" value="Status">
 <attribute name="COLOUR" value="Yellow"/>
 <attribute name="PACKAGE" value="0603"/>
@@
 <attribute name="PACKAGE" value="0402"/>
 </part>
-<part name="JP1" library="SparkFun" deviceset="SMA_EDGE" device="" value="Antenna"/>
+<part name="J1" library="SparkFun" deviceset="SMA_EDGE" device="" value="Antenna"/>
 <part name="GND17" library="supply1" deviceset="GNDA" device="" value="RFGND"/>
 <part name="C1" library="freetronics-master-v1" deviceset="CAP" device="0402" value="22pF">
@@
 </part>
 <part name="G2" library="freetronics-luke" deviceset="GND" device=""/>
-<part name="J1" library="con-molex" deviceset="22-?-04" device="05-7048" value="Interface"/>
 <part name="G3" library="freetronics-luke" deviceset="GND" device=""/>
 <part name="U$4" library="freetronics-luke" deviceset="+3.3V" device=""/>
-<part name="FRAME1" library="frames" deviceset="A4L-LOC" device=""/>
+<part name="FRAME1" library="frames" deviceset="A4L-LOC" device="" value="Frame1"/>
+<part name="J2" library="con-molex" deviceset="22-23-2041" device="" value="Interface"/>
+<part name="SY" library="SparkFun" deviceset="OSHW-LOGO" device="S"/>
 </parts>
 <sheets>
 <sheet>
 <plain>
+<text x="25.4" y="27.94" size="2.54" layer="97">Venus 638FLPX-L GPS Receiver Module</text>
+<text x="45.72" y="22.86" size="2.1844" layer="97">Luke Weston, 2013</text>
+<text x="17.78" y="17.78" size="2.1844" layer="97">http://github.com/lukeweston/SSRPGenericTelemetryModule</text>
+<text x="22.86" y="12.7" size="2.1844" layer="97">Released under the CERN Open Hardware License:</text>
+<text x="43.18" y="7.62" size="2.1844" layer="97">http://ohwr.org/cernohl</text>
 </plain>
 <instances>
@@
 <attribute name="PACKAGE" x="157.48" y="134.62" size="1.27" layer="96"/>
 </instance>
-<instance part="JP1" gate="1" x="160.02" y="127" rot="MR0"/>
+<instance part="J1" gate="1" x="160.02" y="127" rot="MR0"/>
 <instance part="GND17" gate="1" x="165.1" y="109.22" smashed="yes" rot="MR0">
 <attribute name="VALUE" x="162.306" y="106.68" size="1.27" layer="96"/>
@@
 </instance>
 <instance part="G2" gate="G$1" x="88.9" y="104.14" rot="MR0"/>
-<instance part="J1" gate="-1" x="45.72" y="101.6" smashed="yes" rot="MR0">
-<attribute name="NAME" x="38.1" y="101.6" size="1.27" layer="95"/>
-<attribute name="VALUE" x="38.1" y="104.14" size="1.27" layer="96"/>
-</instance>
-<instance part="J1" gate="-2" x="45.72" y="99.06" smashed="yes" rot="MR0">
-<attribute name="NAME" x="38.1" y="99.06" size="1.27" layer="95"/>
-</instance>
-<instance part="J1" gate="-3" x="45.72" y="96.52" smashed="yes" rot="MR0">
-<attribute name="NAME" x="38.1" y="96.52" size="1.27" layer="95"/>
-</instance>
-<instance part="J1" gate="-4" x="45.72" y="93.98" smashed="yes" rot="MR0">
-<attribute name="NAME" x="38.1" y="93.98" size="1.27" layer="95"/>
-</instance>
 <instance part="G3" gate="G$1" x="73.66" y="88.9" rot="MR0"/>
 <instance part="U$4" gate="G$1" x="50.8" y="109.22"/>
 <instance part="FRAME1" gate="G$1" x="0" y="0"/>
+<instance part="J2" gate="-1" x="45.72" y="93.98" smashed="yes" rot="R180">
+<attribute name="NAME" x="38.1" y="93.472" size="1.27" layer="95"/>
+<attribute name="VALUE" x="35.56" y="104.14" size="1.27" layer="96"/>
+</instance>
+<instance part="J2" gate="-2" x="45.72" y="96.52" smashed="yes" rot="R180">
+<attribute name="NAME" x="38.1" y="96.012" size="1.27" layer="95"/>
+</instance>
+<instance part="J2" gate="-3" x="45.72" y="99.06" smashed="yes" rot="R180">
+<attribute name="NAME" x="38.1" y="98.552" size="1.27" layer="95"/>
+</instance>
+<instance part="J2" gate="-4" x="45.72" y="101.6" smashed="yes" rot="R180">
+<attribute name="NAME" x="38.1" y="101.092" size="1.27" layer="95"/>
+</instance>
+<instance part="SY" gate="G$1" x="139.7" y="20.32" smashed="yes"/>
 </instances>
 <busses>
@@
 </segment>
 <segment>
-<pinref part="J1" gate="-2" pin="S"/>
 <wire x1="48.26" y1="99.06" x2="73.66" y2="99.06" width="0.1524" layer="91"/>
 <wire x1="73.66" y1="99.06" x2="73.66" y2="91.44" width="0.1524" layer="91"/>
@@
 <wire x1="73.66" y1="99.06" x2="73.66" y2="101.6" width="0.1524" layer="91"/>
 <junction x="73.66" y="99.06"/>
+<pinref part="J2" gate="-3" pin="S"/>
 </segment>
 </net>
@@
 </segment>
 <segment>
-<pinref part="J1" gate="-1" pin="S"/>
 <wire x1="48.26" y1="101.6" x2="50.8" y2="101.6" width="0.1524" layer="91"/>
 <wire x1="50.8" y1="101.6" x2="50.8" y2="106.68" width="0.1524" layer="91"/>
 <pinref part="U$4" gate="G$1" pin="+3V3"/>
+<pinref part="J2" gate="-4" pin="S"/>
 </segment>
 </net>
 <net name="RFGND" class="0">
 <segment>
-<pinref part="JP1" gate="1" pin="GND@0"/>
+<pinref part="J1" gate="1" pin="GND@0"/>
 <wire x1="162.56" y1="121.92" x2="165.1" y2="121.92" width="0.1524" layer="91"/>
 <pinref part="GND17" gate="1" pin="GNDA"/>
 <wire x1="165.1" y1="121.92" x2="165.1" y2="119.38" width="0.1524" layer="91"/>
 <wire x1="165.1" y1="111.76" x2="165.1" y2="114.3" width="0.1524" layer="91"/>
-<pinref part="JP1" gate="1" pin="GND@3"/>
+<pinref part="J1" gate="1" pin="GND@3"/>
 <wire x1="162.56" y1="114.3" x2="165.1" y2="114.3" width="0.1524" layer="91"/>
 <wire x1="165.1" y1="114.3" x2="165.1" y2="116.84" width="0.1524" layer="91"/>
-<pinref part="JP1" gate="1" pin="GND@2"/>
+<pinref part="J1" gate="1" pin="GND@2"/>
 <wire x1="162.56" y1="116.84" x2="165.1" y2="116.84" width="0.1524" layer="91"/>
 <wire x1="165.1" y1="116.84" x2="165.1" y2="119.38" width="0.1524" layer="91"/>
-<pinref part="JP1" gate="1" pin="GND@1"/>
+<pinref part="J1" gate="1" pin="GND@1"/>
 <wire x1="165.1" y1="119.38" x2="162.56" y2="119.38" width="0.1524" layer="91"/>
 <junction x="165.1" y="119.38"/>
@@
 <junction x="152.4" y="132.08"/>
 <pinref part="L1" gate="G$1" pin="2"/>
-<pinref part="JP1" gate="1" pin="SIGNAL"/>
+<pinref part="J1" gate="1" pin="SIGNAL"/>
 <pinref part="IC1" gate="G$1" pin="RFIN"/>
 </segment>
@@
 <wire x1="109.22" y1="106.68" x2="109.22" y2="96.52" width="0.1524" layer="91"/>
 <wire x1="109.22" y1="96.52" x2="48.26" y2="96.52" width="0.1524" layer="91"/>
-<pinref part="J1" gate="-3" pin="S"/>
+<pinref part="J2" gate="-2" pin="S"/>
 </segment>
 </net>
@@
 <wire x1="111.76" y1="104.14" x2="111.76" y2="93.98" width="0.1524" layer="91"/>
 <wire x1="111.76" y1="93.98" x2="48.26" y2="93.98" width="0.1524" layer="91"/>
-<pinref part="J1" gate="-4" pin="S"/>
-</segment>
-</net>
+<pinref part="J2" gate="-1" pin="S"/>
+</segment>
+</net>
